Commit message: Added Ideal System file that loads quadrotor.urdf and attempts to implement control

File: ConnorWork/quadrotor/quadrotor.urdf (robot description, URDF)
Before this commit: robot simple_quadrotor, 5 links, 4 joints
Links:
- link base_link: mass 0.5 -> 0.48; geometry collision box size=0.20 0.20 0.05; visual box size=0.20 0.20 0.05
- link rotor1: mass None -> 0.005
- link rotor2: mass None -> 0.005
- link rotor3: mass None -> 0.005
- link rotor4: mass None -> 0.005
